File: hardware/handset-rev-a/generated/display.kicad_sch (KiCad schematic)
At the start: 13 parts, among them J26 FH12A-50S-0.5SH(55), Q2 AO3400A

Commit message: feat: advance handset prototype design
Parts:
- removed Q2: AO3400A, Package_TO_SOT_SMD:SOT-23, symbol Transistor_FET:Q_NMOS_GSD
- removed R52, R53, R54, R55: 150 1% 0.1W, Resistor_SMD:R_0603_1608Metric, symbol Device:R
- added C90: 1uF 10% X7R 25V, Capacitor_SMD:C_0603_1608Metric, symbol Device:C
- added R82: 4.99k 1%, Resistor_SMD:R_0402_1005Metric, symbol Device:R
- added U32: CAT4004AHU2-GT3, Handset:CAT4004A_UDFN-8_2x2mm_P0.5mm_EP1x1.73mm, symbol Handset:CAT4004AHU2
Connections:
- net +3V3: no longer C47.1, C48.1, J26.35 (Pin_35), J26.40 (Pin_40), J26.41 (Pin_41), J26.42 (Pin_42), J26.7 (Pin_7), J26.8 (Pin_8), J26.9 (Pin_9)
- net +5V_RF: now also C90.1, U32.8 (VIN)
- net GND: now also C90.2, R82.2, U32.2 (GND), U32.9 (EP)
- net LCD_BL_GATE: now also U32.1 (EN/DIM)
- net LCD_CS: no longer J26.38 (Pin_38)
- net LCD_K1: now also U32.3 (LED1)
- net LCD_K2: now also U32.4 (LED2)
- net LCD_K3: now also U32.5 (LED3)
- net LCD_K4: now also U32.6 (LED4)
- net I2C_SCL renamed PANEL_I2C_SCL
- net I2C_SDA renamed PANEL_I2C_SDA
- net LCD_DC renamed PANEL_LCD_DC
- net LCD_RESET renamed PANEL_LCD_RESET
- net SPI_MISO renamed PANEL_SPI_MISO
- net SPI_MOSI renamed PANEL_SPI_MOSI
- net SPI_SCK renamed PANEL_SPI_SCK
- net TOUCH_IRQ renamed PANEL_TOUCH_IRQ
- net TOUCH_RESET renamed PANEL_TOUCH_RESET
- new net LCD_3V0: C47.1, C48.1, J26.35 (Pin_35), J26.40 (Pin_40), J26.41 (Pin_41), J26.42 (Pin_42), J26.7 (Pin_7), J26.8 (Pin_8), J26.9 (Pin_9)
- new net LCD_BL_RSET: R82.1, U32.7 (RSET)
- new net PANEL_LCD_CS: J26.38 (Pin_38)
Other:
- note added: "CAT4004A: four current sinks, 4.99k sets approx. 15mA/channel. On/off only until dimming timing is qualified. Do not fabricate."
- note added: "EN/DIM: external R57 pull-down retains default off. Initialize U2 GPIO low for >=10ms before enabling. Keep high for full-scale current; do not apply ordinary PWM. RSET gain, current drift, heat and purchased panel remain unqualified."
- note removed: "ER-TFT024IPS-3 connector contract. Verify purchased CTP option, FPC orientation, LED branches and supply tolerances."
- moved on the sheet: C47, C48, C49, R56, R57, R58, R59
