File: hardware/handset-rev-a/generated/protection.kicad_sch (KiCad schematic)
At the start: 15 parts, among them J16 EXPANSION_J16, U14 TPS2553DBVR, U15 TPD4E05U06DQAR, U16 TPD4E05U06DQAR

Commit message: feat: add expansion power and signal control
Parts:
- R42: value 100k -> 10k 1%; MPN (none) -> RC0402FR-0710KL
Connections:
- net +3V3: no longer U14.3 (EN)
- net EXP_CS renamed EXP_SW_CS
- net EXP_IRQ renamed EXP_SW_IRQ
- net I2C_SCL renamed EXP_SW_SCL
- net I2C_SDA renamed EXP_SW_SDA
- net SPI_MISO renamed EXP_SW_MISO
- net SPI_MOSI renamed EXP_SW_MOSI
- net SPI_SCK renamed EXP_SW_SCK
- new net EXP_PWR_EN: U14.3 (EN)
Other:
- note added: "Port signals pass through U34 on expansion-control. U14 EN defaults low; fault drives U33 and the hardware signal interlock. No hot-plug approval."
- note removed: "J16 pin order retained. Switch accessories with power off. TPS2553 limit and ESD path require qualification."
- moved on the sheet: C40, C41, J16, R20, R21, R22, R23, R24, R25, R26, R41, R42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
