File: hardware/handset-rev-a/generated/handset.kicad_pcb (KiCad board)
At the start: 4 copper layers, 66 x 142 mm, 281 parts, among them J1 2053380002, J10 LF_COIL_TUNING_REQUIRED, J16 EXPANSION_J16, J2 PACK_NTC_10K_B3435, J20 LORA_915_ANT, J21 CC1101_915_ANT, J22 GNSS_PASSIVE_ANT, J23 DM3D-SF, J24 TSAL6400_CASE_LED, J25 TSOP38438_CASE_RX, J26 FH12A-50S-0.5SH(55), J3 MEDIA_SPEAKER_DIFFERENTIAL, J4 CALL_AUDIO_FROM_MODEM_ADAPTER, J5 CALL_EARPIECE, J6 CALL_MIC, J7 PIM447_HARNESS_VERIFY, J8 MODEM_ADAPTER_3V3_LOGIC, J9 MODEM_POWER_ADAPTER_REQUIRED, Q1 AO3400A, Q3 AO3400A, Q4 AO3400A, Q5 AO3400A, Q6 AO3401A, Q7 AO3400A, Q8 AO3400A, SW1 1, SW10 10, SW11 11, SW12 12, SW13 13, SW14 14, SW15 15, SW16 16, SW17 MCU_BOOT, SW18 MCU_EN, SW19 POWER, SW2 2, SW3 3, SW4 4, SW5 5, SW6 6, SW7 7, SW8 8, SW9 9, U1 ESP32-S3-WROOM-1-N16R8, U10 TPS61023DRLR, U11 TPS62840DLCR, U12 MAX-M10S-00B-01, U13 ST25R3916B-AQET, U14 TPS2553DBVR, U15 TPD4E05U06DQAR, U16 TPD4E05U06DQAR, U17 TPD4E05U06DQAR, U18 SN74AHCT125PWR, U19 SN74LVC1G17DBVR, U2 TCA8418RTWR, U20 TPS63070RNMR, U21 TPS25200DRVR, U22 TUSB320LAIRWBR, U23 TLV70433DBVR, U24 TCA9536DGKR, U25 STM32G031G8U6, U26 TPS7A0230PDBVR, U27 TCA9800DGKR, U28 TPS7A2030PDBVR, U29 SN74LVC244APWR, U3 BQ25186DLHR, U30 SN74LVC2G125DCUR, U31 TCA9406DCUR, U32 CAT4004AHU2-GT3, U33 TCA9537DGSR, U34 SN74CB3Q3245PWR, U35 SN74HCS10PWR, U36 0900FM15K0039001E, U37 BGS12WN6E6327, U4 SX1262IMLTRT, U5 CC1101RGPR, U6 MAX98357AETE+, U7 TPS63802DLAR, U8 MAX17048G+T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

Commit message: feat: route SX1262 digital interface
Parts:
- R10: moved to F.Cu
- moved R10 12.9 mm to (121.5, 49.0)
- moved R91 2.66 mm to (113.0, 33.5)
Routing:
- net SX_CS: track 0.00 -> 95.6 mm, vias 0 -> 7
- net SX_RESET: track 0.00 -> 44.5 mm, vias 0 -> 7
- net SX_DIO1: track 0.00 -> 42.6 mm, vias 0 -> 5
- net SX_BUSY: track 0.00 -> 41.4 mm, vias 0 -> 5
- net SPI_SCK: track 131.2 -> 160.4 mm, vias 15 -> 18
- net KEY_IRQ: track 113.2 -> 142.1 mm, vias 6 -> 8
- net SPI_MOSI: track 120.2 -> 145.1 mm, vias 11 -> 13
- net +3V3: track 516.9 -> 540.8 mm
- net LCD_3V0: track 120.2 -> 138.8 mm
- net SPI_MISO: track 113.7 -> 126.0 mm, vias 14 -> 16
- net LORA_RF_50R: track 6.34 -> 7.64 mm
- net GND: track 444.7 -> 443.7 mm
- net SX_RF_SW: track 3.36 -> 4.12 mm
