File: hardware/handset-rev-a/generated/radios.kicad_sch (KiCad schematic)
At the start: 9 parts, among them J20 LORA_915_ANT, U4 SX1262IMLTRT

Commit message: feat: add SX1262 TCXO clock circuit
Parts:
- added C94: 100nF 10% X7R 16V, Capacitor_SMD:C_0402_1005Metric, symbol Device:C
- added C95: 10pF 5% C0G 50V, Capacitor_SMD:C_0402_1005Metric, symbol Device:C
- added R90: 220R 1%, Resistor_SMD:R_0402_1005Metric, symbol Device:R
- added Y3: 32MHz TCXO 0.5ppm temp, Handset:ECS_TXO_32CSMV_3225, symbol Handset:ECS_TXO_32CSMV
- U4: symbol RF:SX1262IMLTRT -> Handset:SX1262_TCXO_DIO3Supply
Connections:
- net GND: now also C94.2, Y3.1 (GND1), Y3.2 (GND2)
- net SX_TCXO_PWR: now also C94.1, Y3.4 (VDD)
- net SX_XTA: now also C95.2
- net SX_XTB: no longer names the net of U4.4 (XTB)
- new net SX_TCXO_COUPLED: C95.1, R90.2
- new net SX_TCXO_OUT: R90.1, Y3.3 (OUT)
- no-connect marks 0 -> 1
Other:
- note added: "SX1262 core supply and DIO3-controlled TCXO captured. RF frontend remains incomplete; do not power."
- note added: "SetRegulatorMode(0x01) only in STDBY_RC, after hardware qualification. L12 supplies the core, not the SX1262 high-power PA. PA feed, matching/filter and RF switch are still missing. C10 PA bypass and J20 antenna connection remain provisional."
- note added: "Y3 pads 1/2 = GND, 3 = OUT, 4 = VDD. XTB is intentionally NC. Configure DIO3 for 1.8V; provisional startup allowance 5ms. Confirm TCXO output <=1.2Vpp; no qualified maximum in series data."
- note removed: "DC-DC support captured from Semtech DS rev1.2 Fig14-2 and Table5-3. Clock and RF frontend remain incomplete. Do not power."
- note removed: "SetRegulatorMode(0x01) only in STDBY_RC, after hardware qualification. L12 supplies the core, not the SX1262 high-power PA. TCXO, PA feed, matching/filter and RF switch are still missing. C10 PA bypass and J20 antenna connection remain provisional."
