File: hardware/handset-rev-a/generated/cc-radio.kicad_sch (KiCad schematic)
At the start: 29 parts, among them J21 CC1101_915_ANT, U5 CC1101RGPR, Y2 26MHz CL10pF

Commit message: feat: route CC1101 clock and local supplies
Parts:
- U5: footprint Package_DFN_QFN:Texas_RGP0020D_VQFN-20-1EP_4x4mm_P0.5mm_EP2.7x2.7mm -> Handset:CC1101_RGP20_MaskedThermalVias
Changed lines of the file:
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@@
         (font
           (size 1.1 1.1))))
-    (property "Footprint" "Package_DFN_QFN:Texas_RGP0020D_VQFN-20-1EP_4x4mm_P0.5mm_EP2.7x2.7mm"
+    (property "Footprint" "Handset:CC1101_RGP20_MaskedThermalVias"
       (at 86.36 93.98 0)
       (effects
