File: archive/handset-before-usb-relief/ef24884f9bbb/usb.kicad_sch (KiCad schematic)
At the start: 2 parts, among them U17 TPD4E05U06DQAR

Commit message: fix: clear USB connector hole violations
Parts:
- USB1: footprint Handset:USB4105_GroundCornerRelief -> Connector_USB:USB_C_Receptacle_GCT_USB4105-xx-A_16P_TopMnt_Horizontal
Changed lines of the file:
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@@
         (font
           (size 1.1 1.1))))
-    (property "Footprint" "Handset:USB4105_GroundCornerRelief"
+    (property "Footprint" "Connector_USB:USB_C_Receptacle_GCT_USB4105-xx-A_16P_TopMnt_Horizontal"
       (at 86.36 86.36 0)
       (effects
