File: archive/handset-before-usb-data/2cb4ad59cd64/core.kicad_sch (KiCad schematic)
At the start: 8 parts, among them SW17 MCU_BOOT, SW18 MCU_EN, U1 ESP32-S3-WROOM-1-N16R8

Commit message: feat: route USB data and add termination
Connections:
- net USB_HOST_D_N renamed USB_D_N
- net USB_HOST_D_P renamed USB_D_P
Changed lines of the file:
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@@
       (type default))
 )
-  (global_label "USB_HOST_D_N"
+  (global_label "USB_D_N"
     (shape bidirectional)
     (at 193.04 99.06 180.0)
@@
       (type default))
 )
-  (global_label "USB_HOST_D_P"
+  (global_label "USB_D_P"
     (shape bidirectional)
     (at 193.04 101.6 180.0)
