File: archive/handset-before-sx1262-regulator/e36b11dc7446/handset.kicad_pcb (KiCad board)
At the start: 4 copper layers, 66 x 142 mm, 269 parts, among them J1 2053380002, J10 LF_COIL_TUNING_REQUIRED, J16 EXPANSION_J16, J2 PACK_NTC_10K_B3435, J20 LORA_915_ANT, J21 CC1101_915_ANT, J22 GNSS_PASSIVE_ANT, J23 DM3D-SF, J24 TSAL6400_CASE_LED, J25 TSOP38438_CASE_RX, J26 FH12A-50S-0.5SH(55), J3 MEDIA_SPEAKER_DIFFERENTIAL, J4 CALL_AUDIO_FROM_MODEM_ADAPTER, J5 CALL_EARPIECE, J6 CALL_MIC, J7 PIM447_HARNESS_VERIFY, J8 MODEM_ADAPTER_3V3_LOGIC, J9 MODEM_POWER_ADAPTER_REQUIRED, Q1 AO3400A, Q3 AO3400A, Q4 AO3400A, Q5 AO3400A, Q6 AO3401A, Q7 AO3400A, Q8 AO3400A, SW1 1, SW10 10, SW11 11, SW12 12, SW13 13, SW14 14, SW15 15, SW16 16, SW17 MCU_BOOT, SW18 MCU_EN, SW19 POWER, SW2 2, SW3 3, SW4 4, SW5 5, SW6 6, SW7 7, SW8 8, SW9 9, U1 ESP32-S3-WROOM-1-N16R8, U10 TPS61023DRLR, U11 TPS62840DLCR, U12 MAX-M10S-00B-01, U13 ST25R3916B-AQET, U14 TPS2553DBVR, U15 TPD4E05U06DQAR, U16 TPD4E05U06DQAR, U17 TPD4E05U06DQAR, U18 SN74AHCT125PWR, U19 SN74LVC1G17DBVR, U2 TCA8418RTWR, U20 TPS63070RNMR, U21 TPS25200DRVR, U22 TUSB320LAIRWBR, U23 TLV70433DBVR, U24 TCA9536DGKR, U25 STM32G031G8U6, U26 TPS7A0230PDBVR, U27 TCA9800DGKR, U28 TPS7A2030PDBVR, U29 SN74LVC244APWR, U3 BQ25186DLHR, U30 SN74LVC2G125DCUR, U31 TCA9406DCUR, U32 CAT4004AHU2-GT3, U33 TCA9537DGSR, U34 SN74CB3Q3245PWR, U35 SN74HCS10PWR, U4 SX1262IMLTRT, U5 CC1101RGPR, U6 MAX98357AETE+, U7 TPS63802DLAR, U8 MAX17048G+T, U9 HTRC11001T, Y1 ABM8-27.120MHZ-B2-T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

Commit message: feat: route SX1262 core regulator loop
Parts:
- turned L12 to 0 degrees
Routing:
- net SX_VREG: track 6.73 -> 0.00 mm
- net GND: track 404.5 -> 399.1 mm, vias 175 -> 174
- net SX_DCC_SW: track 2.91 -> 0.00 mm
Changed lines of the file:
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@@
 	(footprint "Inductor_SMD:L_TDK_MLZ2012_h1.25mm"
 		(layer "B.Cu")
-		(at 111 31.5 180)
+		(at 111 31.5)
 		(descr "Inductor, TDK, MLZ2012_h1.25mm, 2.0x1.25x1.25mm, ( \"https://product.tdk.com/system/files/dam/doc/product/inductor/inductor/smd/catalog/inductor_commercial_decoupling_mlz2012_en.pdf\")")
 		(tags "MLZ")
 		(property "Reference" "L12"
-			(at 0 1.58 0)
+			(at 0 1.58 180)
 			(layer "B.Fab")
 			(effects
@@
 		)
 		(property "Value" "15uH 20%"
-			(at 0 -1.58 0)
+			(at 0 -1.58 180)
 			(layer "B.Fab")
 			(hide yes)
@@
 		)
 		(property "Datasheet" ""
-			(at 0 0 0)
+			(at 0 0 180)
 			(layer "B.Fab")
 			(hide yes)
@@
 		)
 		(property "Description" ""
-			(at 0 0 0)
+			(at 0 0 180)
 			(layer "B.Fab")
 			(hide yes)
@@
 		)
 		(property "KiLib_Generator" "inductor/SMD"
-			(at 0 0 0)
+			(at 0 0 180)
 			(layer "B.SilkS")
 			(hide yes)
@@
 		)
 		(property "MPN" "MLZ2012M150WT000"
-			(at 0 0 180)
+			(at 0 0 0)
 			(layer "B.SilkS")
 			(hide yes)
@@
 		(duplicate_pad_numbers_are_jumpers no)
 		(fp_line
-			(start 1.11 -0.86)
-			(end -1.11 -0.86)
+			(start -1.11 0.86)
+			(end 1.11 0.86)
 			(stroke
 				(width 0.12)
@@
 		)
 		(fp_line
-			(start -1.11 0.86)
-			(end 1.11 0.86)
+			(start 1.11 -0.86)
+			(end -1.11 -0.86)
 			(stroke
 				(width 0.12)
@@
 		)
 		(fp_line
-			(start 1.55 0.85)
-			(end 1.55 -0.85)
+			(start -1.55 -0.85)
+			(end -1.55 0.85)
 			(stroke
 				(width 0.05)
@@
 		)
 		(fp_line
-			(start 1.55 -0.85)
-			(end 1.25 -0.85)
+			(start -1.55 0.85)
+			(end -1.25 0.85)
 			(stroke
 				(width 0.05)
@@
 		)
 		(fp_line
-			(start 1.25 0.88)
-			(end 1.25 0.85)
+			(start -1.25 -0.88)
+			(end -1.25 -0.85)
 			(stroke
 				(width 0.05)
@@
 		)
 		(fp_line
-			(start 1.25 0.85)
-			(end 1.55 0.85)
+			(start -1.25 -0.85)
+			(end -1.55 -0.85)
 			(stroke
 				(width 0.05)
@@
 		)
 		(fp_line
-			(start 1.25 -0.85)
-			(end 1.25 -0.88)
+			(start -1.25 0.85)
+			(end -1.25 0.88)
 			(stroke
 				(width 0.05)
@@
 		)
 		(fp_line
-			(start 1.25 -0.88)
-			(end -1.25 -0.88)
+			(start -1.25 0.88)
+			(end 1.25 0.88)
 			(stroke
 				(width 0.05)
@@
 		)
 		(fp_line
-			(start -1.25 0.88)
-			(end 1.25 0.88)
+			(start 1.25 -0.88)
+			(end -1.25 -0.88)
 			(stroke
 				(width 0.05)
@@
 		)
 		(fp_line
-			(start -1.25 0.85)
-			(end -1.25 0.88)
+			(start 1.25 -0.85)
+			(end 1.25 -0.88)
 			(stroke
 				(width 0.05)
@@
 		)
 		(fp_line
-			(start -1.25 -0.85)
-			(end -1.55 -0.85)
+			(start 1.25 0.85)
+			(end 1.55 0.85)
 			(stroke
 				(width 0.05)
@@
 		)
 		(fp_line
-			(start -1.25 -0.88)
-			(end -1.25 -0.85)
+			(start 1.25 0.88)
+			(end 1.25 0.85)
 			(stroke
 				(width 0.05)
@@
 		)
 		(fp_line
-			(start -1.55 0.85)
-			(end -1.25 0.85)
+			(start 1.55 -0.85)
+			(end 1.25 -0.85)
 			(stroke
 				(width 0.05)
@@
 		)
 		(fp_line
-			(start -1.55 -0.85)
-			(end -1.55 0.85)
+			(start 1.55 0.85)
+			(end 1.55 -0.85)
 			(stroke
 				(width 0.05)
@@
 		)
 		(fp_text user "${REFERENCE}"
-			(at 0 0 0)
+			(at 0 0 180)
 			(layer "B.Fab")
 			(effects
@@
 		)
 		(pad "1" smd roundrect
-			(at -0.9 0 180)
+			(at -0.9 0)
 			(size 0.8 1.2)
 			(layers "B.Cu" "B.Mask" "B.Paste")
@@
 		)
 		(pad "2" smd roundrect
-			(at 0.9 0 180)
+			(at 0.9 0)
 			(size 0.8 1.2)
 			(layers "B.Cu" "B.Mask" "B.Paste")
@@
 	)
 	(via
-		(at 108.8 33.5)
-		(size 0.5)
-		(drill 0.3)
-		(layers "F.Cu" "B.Cu")
-		(net "GND")
-	)
-	(via
 		(at 128.4 135.95)
 		(size 0.6)
@@
 	)
 	(segment
-		(start 112.25 34.0625)
-		(end 112.25 35.25)
-		(width 0.25)
-		(layer "B.Cu")
-		(net "GND")
-	)
-	(segment
 		(start 76.5625 83.75)
 		(end 77.4 83.75)
@@
 	)
 	(segment
-		(start 108.78 32.35)
-		(end 108.8 33.5)
-		(width 0.25)
-		(layer "B.Cu")
-		(net "GND")
-	)
-	(segment
 		(start 93 76.75)
 		(end 94 75.75)
@@
 	)
 	(segment
-		(start 111.0625 35.25)
-		(end 112.25 35.25)
-		(width 0.2)
-		(layer "B.Cu")
-		(net "GND")
-	)
-	(segment
 		(start 94.7 44.2)
 		(end 96.9 42)
@@
 	)
 	(segment
-		(start 108.78 31.5)
-		(end 108.78 32.35)
-		(width 0.25)
-		(layer "B.Cu")
-		(net "GND")
-	)
-	(segment
 		(start 96.8 42)
 		(end 96.9 42)
@@
 	)
 	(segment
-		(start 112.25 35.25)
-		(end 113 36)
-		(width 0.25)
-		(layer "B.Cu")
-		(net "GND")
-	)
-	(segment
 		(start 111.55 67.7)
 		(end 111.6 67.65)
@@
 	)
 	(segment
-		(start 107.82 30.98)
-		(end 107.82 31.5)
-		(width 0.25)
-		(layer "B.Cu")
-		(net "SX_VREG")
-	)
-	(segment
-		(start 111.75 34.0625)
-		(end 111.75 33.549999)
-		(width 0.25)
-		(layer "B.Cu")
-		(net "SX_VREG")
-	)
-	(segment
-		(start 110.1 31.9)
-		(end 110.1 31.5)
-		(width 0.25)
-		(layer "B.Cu")
-		(net "SX_VREG")
-	)
-	(segment
-		(start 110.1 31.5)
-		(end 109.6 30.6)
-		(width 0.25)
-		(layer "B.Cu")
-		(net "SX_VREG")
-	)
-	(segment
-		(start 111.75 33.549999)
-		(end 110.1 31.9)
-		(width 0.25)
-		(layer "B.Cu")
-		(net "SX_VREG")
-	)
-	(segment
-		(start 108.2 30.6)
-		(end 107.82 30.98)
-		(width 0.25)
-		(layer "B.Cu")
-		(net "SX_VREG")
-	)
-	(segment
-		(start 109.6 30.6)
-		(end 108.2 30.6)
-		(width 0.25)
-		(layer "B.Cu")
-		(net "SX_VREG")
-	)
-	(segment
 		(start 112.2 39.8)
 		(end 109.91 39.8)
@@
 		(net "CHG_CE_RETURN")
 	)
-	(segment
-		(start 112.75 32.35)
-		(end 111.9 31.5)
-		(width 0.25)
-		(layer "B.Cu")
-		(net "SX_DCC_SW")
-	)
-	(segment
-		(start 112.75 34.0625)
-		(end 112.75 32.35)
-		(width 0.25)
-		(layer "B.Cu")
-		(net "SX_DCC_SW")
-	)
 	(via
