File: archive/handset-before-sx1262-pa/ba78918224a3/radios.kicad_sch (KiCad schematic)
At the start: 25 parts, among them J20 LORA_915_ANT, U36 0900FM15K0039001E, U37 BGS12WN6E6327, U4 SX1262IMLTRT, Y3 32MHz TCXO 0.5ppm temp

Commit message: feat: capture SX1262 PA choke and bypass
Parts:
- removed C101: 47pF 5% C0G 50V, Capacitor_SMD:C_0402_1005Metric, symbol Device:C
- removed L13: 47nH 2%, Inductor_SMD:L_0402_1005Metric, symbol Device:L
- C10: value 47nF 10% X7R 25V -> 100nF; MPN GRM155R71E473KA88D -> (none)
Other:
- note added: "SX1262 clock, supply and RF matching/switch captured. PA feed and RF layout incomplete; do not power."
- note added: "SetRegulatorMode(0x01) only in STDBY_RC, after hardware qualification. L12 supplies the core, not the SX1262 high-power PA. PA choke/bypass and final RF placement/routing remain open. C10 PA bypass and J20 antenna connection remain provisional."
- note removed: "SX1262 clock, supply, PA feed and RF matching/switch captured. RF layout incomplete; do not power."
- note removed: "SetRegulatorMode(0x01) only in STDBY_RC, after hardware qualification. L12 supplies the core, not the SX1262 high-power PA. L13: 47nH PA choke; C10/C101: 47nF/47pF bypass. RAK4270 values; final RF layout and qualification remain open."
- moved on the sheet: C10
